File: electronics/6xv2/cape-servitron/cape-servitron-v1.brd (EAGLE design)
At the start: 160 x 140.6 mm, 100 parts, among them IC1 74541PW, IC2 74541PW, IC3 74541PW, IC4 LM2574M-5.0, M0-CONN PINHEAD-5MM-1X2, M0-CONN1 PINHEAD-5MM-1X2, M0-CONN2 PINHEAD-5MM-1X2, M0-CONN3 PINHEAD-5MM-1X2, M0-CONN4 PINHEAD-5MM-1X2, M0-CONN5 PINHEAD-5MM-1X2, Q1 BSS123

Commit message: added holes, layout mostly done
Parts:
- added H1, H2, H3, H4: MOUNT-HOLE3.0, holes:3,0
- moved BRAKE 273.1 mm to (149.9, 64.8), turned to 90 degrees
- moved D1 249.9 mm to (138.4, 48.3), turned to 180 degrees
- moved POWER_IN 233.1 mm to (149.9, 111.8), turned to 90 degrees
- moved C9 232.1 mm to (114.3, 134.6), turned to 270 degrees
- moved C5 229.5 mm to (124.5, 134.6), turned to 270 degrees
- moved C3 227.4 mm to (111.8, 77.5), turned to 270 degrees
- moved L1 227.3 mm to (116.8, 33.0)
- moved C12 226.5 mm to (73.7, 41.9), turned to 180 degrees
- moved IC4 219.6 mm to (133.3, 38.1)
- moved R57 212.8 mm to (121.9, 54.6), turned to 270 degrees
- moved R56 211.1 mm to (127.0, 47.0), turned to 180 degrees
- moved C11 210.2 mm to (130.8, 21.6), turned to 180 degrees
- moved C10 209.7 mm to (144.8, 31.8), turned to 90 degrees
- moved Q1 206.8 mm to (132.1, 53.3)
- moved U$13 203.4 mm to (138.4, 62.2)
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Connections:
- net N$19: now also U$4.4; no longer U$4.3
- net N$20: now also U$4.3; no longer U$4.4
Routing:
- net GND: track 0.00 -> 308.9 mm, vias 0 -> 13
- net +24V: track 0.00 -> 210.4 mm
- net OUT5A: track 0.00 -> 14.7 mm
- net OUT3A: track 0.00 -> 14.6 mm
- net OUT1A: track 0.00 -> 14.1 mm
- net OUT4B: track 0.00 -> 14.0 mm
- net OUT2B: track 0.00 -> 13.7 mm
- net OUT0B: track 0.00 -> 13.5 mm
- net OUT3B: track 0.00 -> 13.0 mm
- net OUT5B: track 0.00 -> 13.0 mm
- net OUT0A: track 0.00 -> 12.9 mm
- net OUT2A: track 0.00 -> 12.9 mm
- net OUT4A: track 0.00 -> 12.9 mm
- net OUT1B: track 0.00 -> 12.9 mm
- added copper zone on layer 1, net +24V
- added copper zone on layer 1, net OUT0A
- added copper zone on layer 1, net OUT0B
- added copper zone on layer 1, net OUT1A
- added copper zone on layer 1, net OUT1B
- added copper zone on layer 1, net OUT2A
- added copper zone on layer 1, net OUT2B
- added copper zone on layer 1, net OUT3A
- added copper zone on layer 1, net OUT3B
- added copper zone on layer 1, net OUT4A
- added copper zone on layer 1, net OUT4B
- added copper zone on layer 1, net OUT5A
- added copper zone on layer 1, net OUT5B
Other:
- board size 160 x 140.6 mm -> 158.8 x 147.3 mm
